File: Platform/Platform.sch (EAGLE design)
At the start: 37 parts, among them U1 FT232RLSSOP, U2 LM2574N, X1 USBSMD, Y1 RESONATORSMD

Commit message: updates from prototype 3
Parts:
- removed U2: LM2574N, Dustin:LM2574NSOIC8
- added LOGO1: OSHW_LOGO_10MILX0750-NT, ohw-logo:OSHW_LOGO_10MILX0750-NT
- added U$1: LM2594, Dustin:LM2594
- C8: device Dustin:CAP_POLCAP-B -> SparkFun:CAP0805
- LED1, LED2: device SparkFun:LED1206 -> SparkFun:LED0603
- S1: value (none) -> SWITCH-SPDT; device SparkFun:SWITCH-SPSTSMD2 -> Dustin:SWITCH-SPDT
Connections:
- net FTDI-GND: now also C8.2; no longer C8.-
- net FTDI-VCC: now also C8.1; no longer C8.+
- net GNDLINK: now also U$1.ON/OFF, U$1.PWR_GND; no longer U2.ON/OFF, U2.PWR_GND, U2.SIG_GND
- net N$3: now also U$1.OUTPUT; no longer U2.OUTPUT
- net RAW: now also U$1.VIN; no longer U2.VIN
- net VCCLINK: now also U$1.FB; no longer U2.FB
Other:
- note added: "Robotic Minion Starter Kit (Ardunio Compatible) by Dustin Andrews and David Andrews 2012"
- note removed: "Red Soul 16x2 Ardunio Compatible Platform by Dustin Andrews 2012"
Changed lines of the file:
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@@
 <part name="L1" library="SparkFun" deviceset="INDUCTOR" device="0805" value="10uH"/>
 <part name="U$2" library="Dustin" deviceset="EN12-VS11AF" device="TOPKNOB"/>
-<part name="S1" library="SparkFun" deviceset="SWITCH-SPST" device="SMD2"/>
 <part name="R2" library="SparkFun" deviceset="RESISTOR" device="0805-RES" value="220"/>
 <part name="SPI" library="SparkFun" deviceset="AVR_SPI_PRG_6" device="NS"/>
@@
 <part name="C6" library="Dustin" deviceset="CAP_POL" device="" value="0.01uf"/>
 <part name="C9" library="SparkFun" deviceset="CAP" device="0805" value="0.1uf"/>
-<part name="U2" library="Dustin" deviceset="LM2574N" device="SOIC8" value="LM2574N"/>
 <part name="L2" library="SparkFun" deviceset="INDUCTOR" device="0805" value="100uH"/>
 <part name="U$4" library="Dustin" deviceset="DCJACK" device="SMD"/>
 <part name="C4" library="Dustin" deviceset="CAP_POL" device="F80" value="68uf"/>
 <part name="C5" library="Dustin" deviceset="CAP_POL" device="8X10" value="120uf"/>
-<part name="C8" library="Dustin" deviceset="CAP_POL" device="CAP-B" value="4.7uf"/>
 <part name="SCHOTTKEY" library="Dustin" deviceset="DIODE-SCHOTTKY" device="" value=""/>
 <part name="SG2" library="SparkFun" deviceset="BUZZER" device="SMD"/>
-<part name="LED2" library="SparkFun" deviceset="LED" device="1206" value="RED"/>
+<part name="LED2" library="SparkFun" deviceset="LED" device="0603" value="RED"/>
 <part name="R4" library="SparkFun" deviceset="TRIMPOT" device="SMD"/>
 <part name="LCDCON" library="con-harting" deviceset="CON14" device=""/>
-<part name="LED1" library="SparkFun" deviceset="LED" device="1206" value="GRN"/>
+<part name="LED1" library="SparkFun" deviceset="LED" device="0603" value="GRN"/>
 <part name="R3" library="SparkFun" deviceset="RESISTOR" device="0805-RES" value="220"/>
 <part name="LINK1" library="Dustin" deviceset="LINK" device=""/>
@@
 <part name="JP1" library="Dustin" deviceset="M14B" device=""/>
 <part name="C7" library="SparkFun" deviceset="CAP" device="0805" value="0.1uf"/>
+<part name="C8" library="SparkFun" deviceset="CAP" device="0805" value="4.7uf"/>
+<part name="U$1" library="Dustin" deviceset="LM2594" device=""/>
+<part name="LOGO1" library="ohw-logo" deviceset="OSHW_LOGO_10MIL" device="X0750-NT"/>
+<part name="S1" library="Dustin" deviceset="SWITCH-SPDT" device="" value=""/>
 </parts>
 <sheets>
@@
 <rectangle x1="-5.08" y1="114.3" x2="93.98" y2="175.26" layer="209"/>
 <text x="-2.54" y="172.72" size="1.778" layer="210">FTDI</text>
-<text x="-5.08" y="185.42" size="1.778" layer="91">Red Soul 16x2 Ardunio Compatible Platform by Dustin Andrews 2012</text>
+<text x="-5.08" y="185.42" size="1.778" layer="91">Robotic Minion Starter Kit (Ardunio Compatible)  by Dustin Andrews and David Andrews 2012</text>
 <text x="-5.08" y="180.34" size="1.778" layer="91">License: http://creativecommons.org/licenses/by/3.0/</text>
 <rectangle x1="99.06" y1="116.84" x2="220.98" y2="175.26" layer="209"/>
@@
 <instance part="L1" gate="G$1" x="22.86" y="73.66" rot="R180"/>
 <instance part="U$2" gate="G$1" x="208.28" y="76.2"/>
-<instance part="S1" gate="1" x="109.22" y="132.08" rot="R270"/>
 <instance part="R2" gate="G$1" x="241.3" y="93.98" rot="R180"/>
 <instance part="SPI" gate="G$1" x="124.46" y="93.98"/>
@@
 <instance part="C6" gate="C$1" x="20.32" y="162.56" rot="R180"/>
 <instance part="C9" gate="G$1" x="43.18" y="132.08" rot="R90"/>
-<instance part="U2" gate="G$1" x="149.86" y="149.86"/>
 <instance part="L2" gate="G$1" x="175.26" y="144.78" rot="R90"/>
 <instance part="U$4" gate="G$1" x="111.76" y="162.56"/>
 <instance part="C4" gate="C$1" x="134.62" y="134.62"/>
 <instance part="C5" gate="C$1" x="185.42" y="134.62"/>
-<instance part="C8" gate="C$1" x="17.78" y="127"/>
 <instance part="SCHOTTKEY" gate="G$1" x="165.1" y="137.16" rot="R90"/>
 <instance part="SG2" gate="G$1" x="203.2" y="91.44" rot="R90"/>
@@
 <attribute name="VALUE" x="34.036" y="131.699" size="1.778" layer="96" rot="R180"/>
 </instance>
+<instance part="C8" gate="G$1" x="17.78" y="127"/>
+<instance part="U$1" gate="G$1" x="149.86" y="149.86"/>
+<instance part="LOGO1" gate="G$1" x="104.14" y="182.88"/>
+<instance part="S1" gate="G$1" x="109.22" y="129.54" rot="R270"/>
 </instances>
 <busses>
@@
 <net name="RAW" class="0">
 <segment>
-<pinref part="S1" gate="1" pin="O"/>
 <wire x1="111.76" y1="127" x2="121.92" y2="127" width="0.1524" layer="91"/>
 <label x="116.84" y="127" size="1.778" layer="95"/>
-</segment>
-<segment>
-<pinref part="U2" gate="G$1" pin="VIN"/>
+<pinref part="S1" gate="G$1" pin="O"/>
+</segment>
+<segment>
 <wire x1="137.16" y1="157.48" x2="134.62" y2="157.48" width="0.1524" layer="91"/>
 <label x="127" y="157.48" size="1.778" layer="95"/>
@@
 <pinref part="C4" gate="C$1" pin="+"/>
 <junction x="134.62" y="157.48"/>
+<pinref part="U$1" gate="G$1" pin="VIN"/>
 </segment>
 </net>
@@
 <wire x1="106.68" y1="144.78" x2="104.14" y2="144.78" width="0.1524" layer="91"/>
 <wire x1="104.14" y1="144.78" x2="104.14" y2="137.16" width="0.1524" layer="91"/>
-<pinref part="S1" gate="1" pin="P"/>
 <wire x1="109.22" y1="137.16" x2="109.22" y2="134.62" width="0.1524" layer="91"/>
 <pinref part="9V" gate="G$1" pin="1"/>
 <wire x1="119.38" y1="144.78" x2="106.68" y2="144.78" width="0.1524" layer="91"/>
+<pinref part="S1" gate="G$1" pin="P"/>
 </segment>
 <segment>
@@
 <segment>
 <pinref part="L2" gate="G$1" pin="1"/>
-<pinref part="U2" gate="G$1" pin="OUTPUT"/>
 <wire x1="167.64" y1="144.78" x2="165.1" y2="144.78" width="0.1524" layer="91"/>
 <junction x="165.1" y="144.78"/>
@@
 <wire x1="165.1" y1="139.7" x2="165.1" y2="144.78" width="0.1524" layer="91"/>
 <pinref part="SCHOTTKEY" gate="G$1" pin="C"/>
+<pinref part="U$1" gate="G$1" pin="OUTPUT"/>
 </segment>
 </net>
@@
 <junction x="185.42" y="144.78"/>
 <wire x1="185.42" y1="144.78" x2="195.58" y2="144.78" width="0.1524" layer="91"/>
-<pinref part="U2" gate="G$1" pin="FB"/>
 <wire x1="162.56" y1="152.4" x2="185.42" y2="152.4" width="0.1524" layer="91"/>
 <wire x1="185.42" y1="152.4" x2="185.42" y2="144.78" width="0.1524" layer="91"/>
@@
 <pinref part="C5" gate="C$1" pin="+"/>
 <pinref part="LINK1" gate="G$1" pin="P$1"/>
+<pinref part="U$1" gate="G$1" pin="FB"/>
 </segment>
 </net>
@@
 <wire x1="185.42" y1="129.54" x2="185.42" y2="132.08" width="0.1524" layer="91"/>
 <junction x="142.24" y="129.54"/>
-<junction x="144.78" y="129.54"/>
 <junction x="147.32" y="129.54"/>
-<pinref part="U2" gate="G$1" pin="PWR_GND"/>
 <wire x1="142.24" y1="129.54" x2="142.24" y2="139.7" width="0.1524" layer="91"/>
-<pinref part="U2" gate="G$1" pin="SIG_GND"/>
-<wire x1="144.78" y1="129.54" x2="144.78" y2="139.7" width="0.1524" layer="91"/>
-<pinref part="U2" gate="G$1" pin="ON/OFF"/>
 <wire x1="147.32" y1="129.54" x2="147.32" y2="139.7" width="0.1524" layer="91"/>
 <junction x="165.1" y="129.54"/>
@@
 <label x="167.64" y="129.54" size="1.778" layer="95"/>
 <pinref part="LINK2" gate="G$1" pin="P$1"/>
+<pinref part="U$1" gate="G$1" pin="ON/OFF"/>
+<pinref part="U$1" gate="G$1" pin="PWR_GND"/>
 </segment>
 </net>
@@
 <junction x="17.78" y="134.62"/>
 <wire x1="17.78" y1="134.62" x2="-2.54" y2="134.62" width="0.1524" layer="91"/>
-<pinref part="C8" gate="C$1" pin="+"/>
 <wire x1="17.78" y1="132.08" x2="17.78" y2="134.62" width="0.1524" layer="91"/>
 <label x="30.48" y="170.18" size="1.778" layer="95"/>
+<pinref part="C8" gate="G$1" pin="1"/>
 </segment>
 </net>
@@
 <wire x1="38.1" y1="124.46" x2="38.1" y2="132.08" width="0.1524" layer="91"/>
 <label x="27.94" y="121.92" size="1.778" layer="95"/>
-<pinref part="C8" gate="C$1" pin="-"/>
 <wire x1="17.78" y1="121.92" x2="17.78" y2="124.46" width="0.1524" layer="91"/>
 <wire x1="15.24" y1="121.92" x2="17.78" y2="121.92" width="0.1524" layer="91"/>
@@
 <wire x1="10.16" y1="157.48" x2="10.16" y2="154.94" width="0.1524" layer="91"/>
 <junction x="33.02" y="121.92"/>
-</segment>
-</net>
+<pinref part="C8" gate="G$1" pin="2"/>
+</segment>
+</net>

Commit message: prototype 4
Parts:
- LED1, LED2: device SparkFun:LED0603 -> SparkFun:LED0805
- renumbered U$1 to SWITCHREG
Changed lines of the file:
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@@
 <part name="SCHOTTKEY" library="Dustin" deviceset="DIODE-SCHOTTKY" device="" value=""/>
 <part name="SG2" library="SparkFun" deviceset="BUZZER" device="SMD"/>
-<part name="LED2" library="SparkFun" deviceset="LED" device="0603" value="RED"/>
+<part name="LED2" library="SparkFun" deviceset="LED" device="0805" value="RED"/>
 <part name="R4" library="SparkFun" deviceset="TRIMPOT" device="SMD"/>
 <part name="LCDCON" library="con-harting" deviceset="CON14" device=""/>
-<part name="LED1" library="SparkFun" deviceset="LED" device="0603" value="GRN"/>
+<part name="LED1" library="SparkFun" deviceset="LED" device="0805" value="GRN"/>
 <part name="R3" library="SparkFun" deviceset="RESISTOR" device="0805-RES" value="220"/>
 <part name="LINK1" library="Dustin" deviceset="LINK" device=""/>
@@
 <part name="C7" library="SparkFun" deviceset="CAP" device="0805" value="0.1uf"/>
 <part name="C8" library="SparkFun" deviceset="CAP" device="0805" value="4.7uf"/>
-<part name="U$1" library="Dustin" deviceset="LM2594" device=""/>
+<part name="SWITCHREG" library="Dustin" deviceset="LM2594" device=""/>
 <part name="LOGO1" library="ohw-logo" deviceset="OSHW_LOGO_10MIL" device="X0750-NT"/>
 <part name="S1" library="Dustin" deviceset="SWITCH-SPDT" device="" value=""/>
@@
 </instance>
 <instance part="C8" gate="G$1" x="17.78" y="127"/>
-<instance part="U$1" gate="G$1" x="149.86" y="149.86"/>
+<instance part="SWITCHREG" gate="G$1" x="149.86" y="149.86"/>
 <instance part="LOGO1" gate="G$1" x="104.14" y="182.88"/>
 <instance part="S1" gate="G$1" x="109.22" y="129.54" rot="R270"/>
@@
 <pinref part="C4" gate="C$1" pin="+"/>
 <junction x="134.62" y="157.48"/>
-<pinref part="U$1" gate="G$1" pin="VIN"/>
+<pinref part="SWITCHREG" gate="G$1" pin="VIN"/>
 </segment>
 </net>
@@
 <wire x1="165.1" y1="139.7" x2="165.1" y2="144.78" width="0.1524" layer="91"/>
 <pinref part="SCHOTTKEY" gate="G$1" pin="C"/>
-<pinref part="U$1" gate="G$1" pin="OUTPUT"/>
+<pinref part="SWITCHREG" gate="G$1" pin="OUTPUT"/>
 </segment>
 </net>
@@
 <pinref part="C5" gate="C$1" pin="+"/>
 <pinref part="LINK1" gate="G$1" pin="P$1"/>
-<pinref part="U$1" gate="G$1" pin="FB"/>
+<pinref part="SWITCHREG" gate="G$1" pin="FB"/>
 </segment>
 </net>
@@
 <label x="167.64" y="129.54" size="1.778" layer="95"/>
 <pinref part="LINK2" gate="G$1" pin="P$1"/>
-<pinref part="U$1" gate="G$1" pin="ON/OFF"/>
-<pinref part="U$1" gate="G$1" pin="PWR_GND"/>
-</segment>
-</net>
+<pinref part="SWITCHREG" gate="G$1" pin="ON/OFF"/>
+<pinref part="SWITCHREG" gate="G$1" pin="PWR_GND"/>
+</segment>
+</net>
